File: kicad/faema-president.kicad_sch (KiCad schematic)
At the start: 42 parts, among them J1 AC_INPUT, J2 CALDEIRA_2400W, J3 PT100_CALDEIRA, J5 ILI9341_DISP, J6 PT100_GRUPO, J7 SONDA_NIVEL, J8 PRESET_BTNS, J9 ENCODER, Q1 2N7002, U1 ESP32-S3 Mini, U2 HLK-PM05, U3 AMS1117-3.3, U4 MAX31865_CALDEIRA, U5 DS3231, U6 MAX31865_GRUPO

Commit message: modificações feita pelo Codex na geração do esquematico
Connections:
- net +3V3: now also U4.9 (GND), U5.4 (GND), U6.9 (GND)
- net +5V: now also R7.2, U2.4 (GND); no longer R7.1
- net BTN3: now also U1.21 (GPIO21/BTN3)
- net CS_MAX_GRUPO: now also U1.18 (GPIO18/CS_MAX2)
- net FORCE_PLUS_U4: now also J3.4
- net FORCE_PLUS_U6: now also J6.4
- net GND: now also BT1.1, J7.1, R10.1, R9.1, U2.3 (+5V), U4.1 (VDD), U5.2 (VCC), U6.1 (VDD); no longer R9.2
- net I2C_SCL: now also U5.1 (32K)
- net LED_STATUS: now also D1.1 (A), U1.24 (USB_D-)
- net LEVEL_SENSE: now also J7.2, R11.2
- net L_FUSED: now also U2.2 (AC_N)
- net L_IN: now also J1.3
- net MAX_DRDY: now also U1.25 (EN)
- net N_IN: now also J1.2, J2.1, U2.1 (AC_L)
- net Q1_GATE: now also R9.2; no longer Q1.1 (G)
- net RTDIN_MINUS_U4: now also J3.2
- net RTDIN_MINUS_U6: now also J6.2
- net RTDIN_PLUS_U4: now also J3.3
- net RTDIN_PLUS_U6: now also J6.3
- net SSR_CTRL: now also R_gate.1
- net SSR_MINUS: now also Q1.3 (S), SSR1.3 (CTRL+)
- net SSR_PLUS: now also R7.1, SSR1.4 (CTRL-)
- net PE: now reaches J1.1
- net AC_SSR_L_OUT: now reaches SSR1.1 (AC1)
- net AC_SSR_L_OUT: now also J2.2
- net AC_SSR_L_IN: now reaches SSR1.2 (AC2)
- net REFIN_MINUS_U4: now reaches U4.13 (REFIN-)
- net REFIN_MINUS_U6: now reaches U6.13 (REFIN-)
- net FORCE_MINUS_U4: now reaches J3.1
- net FORCE_MINUS_U6: now reaches J6.1
- net VBAT_RTC: now reaches BT1.2
Other:
- note added: "DISPLAY / UI"
- note added: "DRIVE SSR / SEGURANÇA"
- note added: "ENTRADA AC / PROTEÇÕES"
- note added: "FAEMA PRESIDENT - Rev.5 Esquemático reorganizado por blocos funcionais."
- note added: "FONTE 5V / 3V3"
- note added: "MCU / CONTROLE"
- note added: "R9: pull-down de segurança Q1 desliga o SSR por low-side."
- note added: "RTC"
- note added: "SENSOR PT100 CALDEIRA"
- note added: "SENSOR PT100 GRUPO"
- note removed: "FAEMA PRESIDENT - Rev.5 Conectar nets com mesmo nome global label. Ver CLAUDE.md para especificação completa."
- note removed: "MCU"
- note removed: "PERIFÉRICOS"
- note removed: "R9: PULL-DOWN SEGURANÇA Garante SSR OFF durante boot"
- note removed: "REGULAÇÃO DC 5V → 3.3V"
- note removed: "SENSORES PT100"
- note removed: "SEÇÃO AC 220VAC"
- moved on the sheet: BT1, C1, C10, C11, C12, C2, C3, C4, C7, C8, C9, D1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
